File: EEGFrontier.kicad_pcb (KiCad board)
At the start: 2 copper layers, 55 x 41.5 mm, 33 parts, among them J1 Conn_01x08_Pin, SW1 SW_Push, U1 102010428, U2 ADS1299-4PAGR

Commit message: Refactor code structure for improved readability and maintainability
Parts:
- J1: footprint Connector_PinHeader_2.54mm:PinHeader_1x08_P2.54mm_Vertical -> Connector_PinHeader_2.54mm:PinHeader_1x08_P2.54mm_Horizontal
