File: EEGFrontier.kicad_sch (KiCad schematic)
At the start: 29 parts, among them J1 Conn_01x08_Pin, SW1 SW_Push, U1 102010428, U2 ADS1299-4PAGR

Commit message: Refactor code structure for improved readability and maintainability
Parts:
- J1: footprint Connector_PinHeader_2.54mm:PinHeader_1x08_P2.54mm_Vertical -> Connector_PinHeader_2.54mm:PinHeader_1x08_P2.54mm_Horizontal
Changed lines of the file:
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@@
 			)
 		)
-		(property "Footprint" "Connector_PinHeader_2.54mm:PinHeader_1x08_P2.54mm_Vertical"
+		(property "Footprint" "Connector_PinHeader_2.54mm:PinHeader_1x08_P2.54mm_Horizontal"
 			(at 190.5 93.98 0)
 			(effects
